File: GripperGoFa_ArduinoNano.kicad_sch (KiCad schematic)
At the start: 16 parts, among them J1 Conn_01x02, J2 Conn_01x04, J3 Conn_01x03, J4 Conn_01x05, J5 Conn_01x02, U1 HCPL-2631, U2 HCPL-2631

Commit message: update components
Parts:
- removed R5, R6: 2k7, Resistor_SMD:R_1210_3225Metric, symbol Device:R
- removed U2: HCPL-2631, Package_DIP:DIP-8_W7.62mm, symbol Isolator:HCPL-2631
- added D1: D, symbol Device:D
- added J6: Magnet, Connector_PinSocket_2.54mm:PinSocket_1x02_P2.54mm_Vertical, symbol Connector_Generic:Conn_01x02
- added K1: SRD-05VDC-SL-C, Relay_THT:RELAY_SRD-05VDC-SL-C, symbol SRD-05VDC-SL-C:SRD-05VDC-SL-C
- added R7: R, Resistor_SMD:R_1210_3225Metric_Pad1.30x2.65mm_HandSolder, symbol Device:R
- J1: value Conn_01x02 -> VCC
- J2: value Conn_01x04 -> Input
- J3: value Conn_01x03 -> Servo
- J4: value Conn_01x05 -> OptSensor
- J5: value Conn_01x02 -> FSR
Connections:
- net +24V: now also D1.2 (A)
- net GND: now also J6.2 (Pin_2), K1.A2, R7.2
- net at A1.21 (A2), J5.2 (Pin_2): now also R7.1
- net D6: no longer names the net of A1.9 (D6)
- net D7 renamed MagnetDO
- net MagnetDO: now also K1.A1
- new net: J6.1 (Pin_1), K1.COM
- new net: D1.1 (K), K1.NO
Other:
- moved on the sheet: C1, J3
