File: XIAO_RP2040/gripper_xiao2040.kicad_sch (KiCad schematic)
At the start: 16 parts, among them J1 GoFa IO, J2 VGoFa, J3 Servo, J4 Magnet, J5 Conn_01x04, U1 XIAO-RP2040-DIP, U2 HCPL-2631

Commit message: PCB design complete and built. Arduino code still testing
Parts:
- added C3: C, Capacitor_SMD:C_1210_3225Metric, symbol Device:C
- added IC1: INA236BIDDFR, SOT65P280X110-8N, symbol INA236:INA236BIDDFR
- added J6: Jumper, Connector_PinHeader_1.27mm:PinHeader_1x03_P1.27mm_Vertical, symbol Connector_Generic:Conn_01x03
- added Q1: BC237, Package_TO_SOT_THT:TO-92_Inline, symbol Transistor_BJT:BC237
- added R7, R8: 2K7, Resistor_SMD:R_1210_3225Metric, symbol Device:R
- added Rshunt1: R, Resistor_SMD:R_1210_3225Metric, symbol Device:R
- D1: footprint Diode_THT:D_DO-35_SOD27_P7.62mm_Horizontal -> Diode_SMD:Nexperia_CFP3_SOD-123W
- J1, J4: footprint Connector_PinHeader_2.54mm:PinHeader_1x02_P2.54mm_Vertical -> TerminalBlock_Phoenix:TerminalBlock_Phoenix_MPT-0,5-2-2.54_1x02_P2.54mm_Horizontal
- J2: footprint Connector_PinSocket_2.54mm:PinSocket_1x02_P2.54mm_Vertical -> TerminalBlock_Phoenix:TerminalBlock_Phoenix_MPT-0,5-2-2.54_1x02_P2.54mm_Horizontal
- J3: footprint Connector_PinHeader_2.54mm:PinHeader_1x03_P2.54mm_Vertical -> Connector_PinHeader_2.54mm:PinHeader_1x03_P2.54mm_Horizontal
- R1, R2, R3, R5: value R -> 2K7
- R4: value R -> 4K7
Connections:
- net +3V: now also C3.2, IC1.4 (VS), R7.2, R8.1
- net +5V: now also IC1.1 (IN+), Rshunt1.2; no longer J3.2 (Pin_2)
- net DO2: now also J6.2 (Pin_2); no longer R2.2, R4.1
- net GND: now also J2.1 (Pin_1), C3.1, IC1.3 (GND), Q1.3 (E); no longer D1.2 (A), J2.2 (Pin_2), J4.2 (Pin_2)
- net do1_coupled: now also U1.9 (GPIO2/SCK); no longer U1.10 (GPIO4/MISO)
- net do2_coupled: now also U1.10 (GPIO4/MISO); no longer U1.9 (GPIO2/SCK)
- net SDA: now reaches U1.5 (GPIO6/SDA)
- net SDA: now also IC1.6 (SDA), R8.2
- net SCL: now reaches U1.6 (GPIO7/SCL)
- net SCL: now also IC1.5 (SCL), R7.1
- net Vcc renamed VGoFa
- net VGoFa: now also D1.1 (K), J2.2 (Pin_2), J4.2 (Pin_2); no longer J2.1 (Pin_1)
- new net: D1.2 (A), J4.1 (Pin_1), Q1.1 (C)
- new net: Q1.2 (B), R4.2
- new net: J6.1 (Pin_1), R2.2
- new net: J6.3 (Pin_3), R4.1
- new net Vsensed: IC1.2 (IN-), J3.2 (Pin_2), Rshunt1.1
Other:
- moved on the sheet: J1, J2, R4
